Commit message: speed up simulate by remove collision in urdf model

File: src/tandem_mani/urdf/tandem_mani_no_collision.urdf (robot description, URDF)
Before this commit: robot tandem_mani, 6 links, 5 joints
Links:
- link base_link: geometry visual mesh filename=package://tandem_mani/meshes/base_link.STL
- link link1: geometry visual mesh filename=package://tandem_mani/meshes/link1.STL
- link link2: geometry visual mesh filename=package://tandem_mani/meshes/link2.STL
- link link3: geometry visual mesh filename=package://tandem_mani/meshes/link3.STL
- link link4: geometry visual mesh filename=package://tandem_mani/meshes/link4.STL

Commit message: try to add collision but oscillation

File: src/tandem_mani/urdf/tandem_mani_no_collision.urdf (robot description, URDF)
Before this commit: robot tandem_mani, 6 links, 5 joints
Links:
- link base_link: geometry collision mesh filename=package://tandem_mani/meshes/base_link_no_collision.STL; visual mesh filename=package://tandem_mani/meshes/base_link.STL
- link link1: geometry collision mesh filename=package://tandem_mani/meshes/link1_no_collision.STL; visual mesh filename=package://tandem_mani/meshes/link1.STL
- link link2: geometry collision mesh filename=package://tandem_mani/meshes/link2_no_collision.STL; visual mesh filename=package://tandem_mani/meshes/link2.STL
- link link3: geometry collision mesh filename=package://tandem_mani/meshes/link3_no_collision.STL; visual mesh filename=package://tandem_mani/meshes/link3.STL
- link link4: geometry collision mesh filename=package://tandem_mani/meshes/link4_no_collision.STL; visual mesh filename=package://tandem_mani/meshes/link4.STL
