Commit message: fix tandem_manipulator and can work fluently

File: src/tandem_mani/urdf/tandem_mani.urdf (robot description, URDF)
Before this commit: robot tandem_mani_1, 6 links, 5 joints
Links:
- removed link link_1
- removed link link_2
- removed link link_3
- removed link link_4
- added link link1, mass 0.2; collision mesh filename=package://tandem_mani/meshes/link1.STL; visual mesh filename=package://tandem_mani/meshes/link1.STL
- added link link2, mass 0.2; collision mesh filename=package://tandem_mani/meshes/link2.STL; visual mesh filename=package://tandem_mani/meshes/link2.STL
- added link link3, mass 0.2; collision mesh filename=package://tandem_mani/meshes/link3.STL; visual mesh filename=package://tandem_mani/meshes/link3.STL
- added link link4, mass 0.2; collision mesh filename=package://tandem_mani/meshes/link4.STL; visual mesh filename=package://tandem_mani/meshes/link4.STL
- link base_link: mass 0.14451 -> 0.2; geometry collision mesh filename=package://tandem_mani/meshes/base_link.STL; visual mesh filename=package://tandem_mani/meshes/base_link.STL
Joints:
- removed joint joint_1
- removed joint joint_2
- removed joint joint_3
- removed joint joint_4
- added joint joint1: type revolute, parent base_link, child link1, origin xyz=-0.00015771 -0.0416 6.4042E-05 rpy=0 0 0, axis 0 1 0, limit lower=-3 upper=3 effort=100 velocity=100
- added joint joint2: type revolute, parent link1, child link2, origin xyz=0.0072805 -0.0512 -0.028071 rpy=0 0 0, axis 0.25105 0 -0.96797, limit lower=-3 upper=3 effort=100 velocity=100
- added joint joint3: type revolute, parent link2, child link3, origin xyz=-0.075777 -0.059106 0.0097896 rpy=0 0 0, axis 0.74347 0.64037 0.19282, limit lower=-3 upper=3 effort=100 velocity=100
- added joint joint4: type revolute, parent link3, child link4, origin xyz=-0.073088 -0.052111 -0.04559 rpy=0 0 0, axis -0.046828 0.33747 -0.94017, limit lower=-3 upper=3 effort=100 velocity=100

Commit message: add .start.sh and change dt param but cannot speed up gazebo

File: src/tandem_mani/urdf/tandem_mani.urdf (robot description, URDF)
Before this commit: robot tandem_mani, 6 links, 5 joints
Joints:
- joint joint1: origin xyz=-0.00015771 -0.0416 6.4042E-05 rpy=0 0 0 -> xyz=-0.00015771 -0.0416 0 rpy=0 0 0

Commit message: set the right initial position

File: src/tandem_mani/urdf/tandem_mani.urdf (robot description, URDF)
Before this commit: robot tandem_mani, 6 links, 5 joints
Links:
- link base_link: mass 0.2 -> 0.14451
- link link1: mass 0.2 -> 0.11786
- link link2: mass 0.2 -> 0.086527
- link link3: mass 0.2 -> 0.1099
- link link4: mass 0.2 -> 0.12676
Joints:
- joint joint1: origin xyz=-0.00015771 -0.0416 0 rpy=0 0 0 -> xyz=-0.00015771 -0.0416 6.4042E-05 rpy=0 0 0
- joint joint2: axis 0.25105 0 -0.96797 -> 0 0 -1; origin xyz=0.0072805 -0.0512 -0.028071 rpy=0 0 0 -> xyz=0 -0.0512 -0.029 rpy=0 0 0
- joint joint3: axis 0.74347 0.64037 0.19282 -> 1 0 0; origin xyz=-0.075777 -0.059106 0.0097896 rpy=0 0 0 -> xyz=-0.0923 0 0.0285 rpy=0 0 0
- joint joint4: axis -0.046828 0.33747 -0.94017 -> 0 0 -1; origin xyz=-0.073088 -0.052111 -0.04559 rpy=0 0 0 -> xyz=-0.0965 0 -0.0287 rpy=0 0 0

File: src/tandem_mani/urdf/tandem_mani_no_collision.urdf (robot description, URDF)
Before this commit: robot tandem_mani, 6 links, 5 joints
Joints:
- joint joint2: axis 0.25105 0 -0.96797 -> 0 0 -1; origin xyz=0.0072805 -0.0512 -0.028071 rpy=0 0 0 -> xyz=0 -0.0512 -0.029 rpy=0 0 0
- joint joint3: axis 0.74347 0.64037 0.19282 -> 1 0 0; origin xyz=-0.075777 -0.059106 0.0097896 rpy=0 0 0 -> xyz=-0.0923 0 0.0285 rpy=0 0 0
- joint joint4: axis -0.046828 0.33747 -0.94017 -> 0 0 -1; origin xyz=-0.073088 -0.052111 -0.04559 rpy=0 0 0 -> xyz=-0.0965 0 -0.0287 rpy=0 0 0

Commit message: add simple collision and works good

File: src/tandem_mani/urdf/tandem_mani.urdf (robot description, URDF)
Before this commit: robot tandem_mani, 6 links, 5 joints
Links:
- link base_link: mass 0.14451 -> 0.2; geometry collision mesh filename=package://tandem_mani/meshes/base_link_no_collision.STL; visual mesh filename=package://tandem_mani/meshes/base_link.STL
- link link1: mass 0.11786 -> 0.2; geometry collision mesh filename=package://tandem_mani/meshes/link1_no_collision.STL; visual mesh filename=package://tandem_mani/meshes/link1.STL
- link link2: mass 0.086527 -> 0.2; geometry collision mesh filename=package://tandem_mani/meshes/link2_no_collision.STL; visual mesh filename=package://tandem_mani/meshes/link2.STL
- link link3: mass 0.1099 -> 0.2; geometry collision mesh filename=package://tandem_mani/meshes/link3_no_collision.STL; visual mesh filename=package://tandem_mani/meshes/link3.STL
- link link4: mass 0.12676 -> 0.2; geometry collision mesh filename=package://tandem_mani/meshes/link4_no_collision.STL; visual mesh filename=package://tandem_mani/meshes/link4.STL
Joints:
- joint joint1: origin xyz=-0.00015771 -0.0416 6.4042E-05 rpy=0 0 0 -> xyz=-0.00015771 -0.0416 0 rpy=0 0 0

Commit message: :sparkles: add fifth link and delete vicon folder

File: src/tandem_mani/urdf/tandem_mani.urdf (robot description, URDF)
Before this commit: robot tandem_mani, 6 links, 5 joints
Links:
- added link link5, mass 0.038763224507172; collision mesh filename=package://tandem_mani/meshes/link5.STL; visual mesh filename=package://tandem_mani/meshes/link5.STL
Joints:
- added joint joint5: type revolute, parent link4, child link5, origin xyz=-0.157 0 0.0587 rpy=0 0 0, axis 0 0 -1, limit lower=0 upper=0 effort=0 velocity=0

Commit message: :sparkles: add platform in tandem_mani.urdf

File: src/tandem_mani/urdf/tandem_mani.urdf (robot description, URDF)
Before this commit: robot tandem_mani, 7 links, 6 joints
Links:
- removed link world
- added link platform, mass 6; collision box size=0.3 0.3 0.1; visual box size=0.3 0.3 0.1
Joints:
- joint joint_fix: origin xyz=-0 -0 0 rpy=-1.5708 0 0 -> xyz=-0 -0 0.05 rpy=-1.5708 0 0; parent world -> platform

Commit message: modify client

File: src/tandem_mani/urdf/tandem_mani.urdf (robot description, URDF)
Before this commit: robot tandem_mani, 7 links, 6 joints
Links:
- removed link platform
- added link link6, mass 0.00001; collision box size=0.1 0.1 0.1; visual box size=0.1 0.1 0.1
- added link world
Joints:
- removed joint joint_fix
- added joint joint6: type fixed, parent link5, child link6, origin xyz=0 0.1 0 rpy=0 1.57079633 1.57079633
- added joint world_joint: type fixed, parent world, child base_link, origin xyz=0 0 1.5 rpy=1.57079633  0 -1.57079633
- joint joint1: origin xyz=-0.00015771 -0.0416 0 rpy=0 0 0 -> xyz=0 -0.0416 0 rpy=0 0 0
- joint joint2: origin xyz=0 -0.0512 -0.029 rpy=0 0 0 -> xyz=0 -0.0512 0 rpy=0 0 0
- joint joint3: axis 1 0 0 -> -1 0 0; origin xyz=-0.0923 0 0.0285 rpy=0 0 0 -> xyz=-0.0923 0 0 rpy=0 0 0
- joint joint4: origin xyz=-0.0965 0 -0.0287 rpy=0 0 0 -> xyz=-0.0965 0 0 rpy=0 0 0
- joint joint5: origin xyz=-0.157 0 0.0587 rpy=0 0 0 -> xyz=-0.157 0 0 rpy=0 0 3.14159265359

Commit message: :sparkles: fix client bug

File: src/tandem_mani/urdf/tandem_mani.urdf (robot description, URDF)
Before this commit: robot tandem_mani, 8 links, 7 joints
Links:
- link base_link: geometry collision mesh filename=package://tandem_mani/meshes/base_link.STL; visual mesh filename=package://tandem_mani/meshes/base_link.STL
- link link1: geometry collision mesh filename=package://tandem_mani/meshes/link1.STL; visual mesh filename=package://tandem_mani/meshes/link1.STL
- link link2: geometry collision mesh filename=package://tandem_mani/meshes/link2.STL; visual mesh filename=package://tandem_mani/meshes/link2.STL
- link link3: geometry collision mesh filename=package://tandem_mani/meshes/link3.STL; visual mesh filename=package://tandem_mani/meshes/link3.STL
- link link4: geometry collision mesh filename=package://tandem_mani/meshes/link4.STL; visual mesh filename=package://tandem_mani/meshes/link4.STL

Commit message: :sparkles: add the new tandem_mani model

File: src/tandem_mani/urdf/tandem_mani.urdf (robot description, URDF)
Before this commit: robot tandem_mani, 8 links, 7 joints
Links:
- removed link link6
- removed link world
- added link end_point, mass 0.000333382798127531; collision mesh filename=package://tandem_mani/meshes/end_point.STL; visual mesh filename=package://tandem_mani/meshes/end_point.STL
- link base_link: mass 0.2 -> 0.285969725659351
- link link1: mass 0.2 -> 0.244953972348195
- link link2: mass 0.2 -> 0.23012452247972
- link link3: mass 0.2 -> 0.249723164589436
- link link4: mass 0.2 -> 0.254533013461218
- link link5: mass 0.038763224507172 -> 0.0494024336689589
Joints:
- removed joint joint6
- removed joint world_joint
- added joint end_joint: type continuous, parent link5, child end_point, origin xyz=0 -0.12 -0.0005 rpy=0.4431 -1.5708 -2.0139, axis 0 0 -1
- joint joint1: axis 0 1 0 -> 0 0 1; limit lower=-30 upper=30 effort=100 velocity=100 -> (none); origin xyz=0 -0.0416 0 rpy=0 0 0 -> xyz=0.00015793 6.4042E-05 -0.093 rpy=0 0 1.5708; type revolute -> continuous
- joint joint2: axis 0 0 -1 -> 0 0 1; limit lower=-30 upper=30 effort=100 velocity=100 -> (none); origin xyz=0 -0.0512 0 rpy=0 0 0 -> xyz=0 0 0 rpy=1.5708 -1.5708 0; type revolute -> continuous
- joint joint3: axis -1 0 0 -> 0 0 -1; limit lower=-30 upper=30 effort=100 velocity=100 -> (none); origin xyz=-0.0923 0 0 rpy=0 0 0 -> xyz=0 -0.189 0 rpy=1.5708 0 0; type revolute -> continuous
- joint joint4: axis 0 0 -1 -> 0 0 1; limit lower=-30 upper=30 effort=100 velocity=100 -> (none); origin xyz=-0.0965 0 0 rpy=0 0 0 -> xyz=0 0 0 rpy=-2.5873 -1.5708 0.98904; type revolute -> continuous
- joint joint5: axis 0 0 -1 -> 0 0 1; limit lower=0 upper=0 effort=0 velocity=0 -> (none); origin xyz=-0.157 0 0 rpy=0 0 3.14159265359 -> xyz=0.157 0 0 rpy=0 0 0; type revolute -> continuous

Commit message: :sparkles: fix tandem_mani model frame

File: src/tandem_mani/urdf/tandem_mani.urdf (robot description, URDF)
Before this commit: robot tandem_mani, 7 links, 6 joints
Joints:
- joint end_joint: axis 0 0 -1 -> 0 0 0; origin xyz=0 -0.12 -0.0005 rpy=0.4431 -1.5708 -2.0139 -> xyz=0 -0.12 -0.0005 rpy=-1.5708 -1.5708 0; type continuous -> fixed
- joint joint4: origin xyz=0 0 0 rpy=-2.5873 -1.5708 0.98904 -> xyz=0 0 0 rpy=-1.5708 -1.5708 0
