Commit message: new controller

File: src/tandem_mani/urdf/tandem_mani_fix.urdf (robot description, URDF)
Before this commit: robot tandem_mani, 8 links, 7 joints
Joints:
- joint joint1: type continuous -> fixed
- joint joint2: type continuous -> fixed
- joint joint3: type continuous -> fixed
- joint joint4: type continuous -> fixed
- joint joint5: type continuous -> fixed
