Commit message: controllor1

File: src/tandem_mani/urdf/tandem_mani1.urdf (robot description, URDF)
Before this commit: robot tandem_mani, 8 links, 7 joints
Links:
- link base_link: mass 0.285969725659351 -> 2
- link end_point: mass 0.000333382798127531 -> 0.000001
- link link1: mass 0.244953972348195 -> 2
- link link2: mass 0.23012452247972 -> 2
- link link3: mass 0.249723164589436 -> 2
- link link4: mass 0.254533013461218 -> 2
- link link5: mass 0.0494024336689589 -> 2
Joints:
- joint end_joint: limit lower=-0.001 upper=0.001 effort=30 velocity=1.0 -> lower=-0.001 upper=0.001 effort=30 velocity=1
- joint joint1: limit lower=-3.14 upper=3.14 effort=30 velocity=10 -> lower=-3.14 upper=3.14 effort=500 velocity=100
- joint joint2: limit lower=-1.5708 upper=1.5708 effort=30 velocity=10 -> lower=-3.14 upper=3.14 effort=500 velocity=100
- joint joint3: limit lower=-3.14 upper=3.14 effort=30 velocity=10 -> lower=-3.14 upper=3.14 effort=500 velocity=100
- joint joint4: limit lower=-1.5708 upper=1.5708 effort=30 velocity=10 -> lower=-3.14 upper=3.14 effort=500 velocity=100
- joint joint5: limit lower=-3.14 upper=3.14 effort=30 velocity=10 -> lower=-3.14 upper=3.14 effort=500 velocity=100
